Commit message: Harden navigation, control FSM, and comms transaction apply

File: ros_ws/cat_follow_bringup/urdf/picarx_lidar.urdf (robot description, URDF)
Before this commit: robot picarx_lidar, 4 links, 3 joints
Links:
- added link ultrasonic_link
Joints:
- added joint base_to_ultrasonic: type fixed, parent base_link, child ultrasonic_link, origin xyz=0.125 0.0 0.04 rpy=0 0 0
